File: Node_F4_V.1.6.kicad_pcb (KiCad board)
At the start: 2 copper layers, 97.5 x 59 mm, 178 parts, among them IC2 MP1584EN, J1 Conn_Jack-DC, J2 Conn_01x10, J3 Conn_01x16_Female, J4 RF_IPEX_U.FL-R-SMT, J5 SWD, J6 WiFi_Prog, J7 RS485, J8 LoRa_Anten, Q1 P_Mosfet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

Commit message: Add via tranh cuon cam va lora
Parts:
- moved F1 3.44 mm to (161.2, 108.0)
- moved D8 2.15 mm to (166.4, 101.0)
- moved L2 2.10 mm to (165.9, 95.7)
- moved C18 1.72 mm to (161.8, 89.1)
- moved C16 1.72 mm to (168.2, 89.1)
- moved C17 1.72 mm to (165.0, 89.1)
- moved R20 1.57 mm to (156.9, 91.7), turned to 180 degrees
- moved C14 1.36 mm to (162.0, 101.0)
- moved JP2 0.41 mm to (158.3, 88.3)
- moved D5 0.22 mm to (151.5, 107.7)
- moved IC2 0.14 mm to (158.4, 99.2)
- moved RV1 0.05 mm to (153.1, 111.8)
Routing:
- net +3.3V: track 507.4 -> 508.9 mm
- net Net-(IC2-BST): track 2.68 -> 1.72 mm
- net GND: vias 181 -> 198

Commit message: Layout nguon
Parts:
- moved C44 1.98 mm to (92.5, 74.8), turned to 135 degrees
- moved C38 1.90 mm to (95.3, 71.0)
- moved R45 1.89 mm to (94.3, 72.0)
- moved C40 1.87 mm to (93.3, 73.0)
- moved C43 1.18 mm to (96.3, 78.3), turned to -45 degrees
- moved C45 1.16 mm to (95.5, 75.2)
- moved C46 1.16 mm to (97.5, 77.2)
- moved Y2 1.16 mm to (98.6, 74.3)
- moved J4 0.49 mm to (82.9, 69.7)
- moved C51 0.37 mm to (85.8, 71.4)
- moved L4 0.28 mm to (87.0, 73.5)
- moved C47 0.26 mm to (94.6, 80.9)
- moved C39 0.22 mm to (89.1, 74.7)
- moved C10 0.17 mm to (90.2, 72.5)
Routing:
- net VCC: track 27.4 -> 13.0 mm
- net +3.3V: track 508.9 -> 503.5 mm, vias 24 -> 25
- net Net-(U6-CAP1): track 5.72 -> 8.25 mm
- net Net-(U6-CAP2): track 3.85 -> 5.95 mm
- net /RS485_DERE: track 8.76 -> 10.5 mm
- net /SWP_SD3: track 23.4 -> 21.7 mm
- net /RS485_RO: track 13.7 -> 15.3 mm
- net Net-(U6-XTAL_N): track 10.9 -> 9.78 mm
- net /RS485_DI: track 9.41 -> 10.4 mm
- net Net-(U6-XTAL_P): track 8.19 -> 7.31 mm
- net /SCK_CLK: track 7.43 -> 6.58 mm
- net Net-(U3-NRST): track 58.2 -> 58.8 mm
- net Net-(U6-U0TXD): track 16.5 -> 16.0 mm
- net Net-(D18-A1): track 16.0 -> 16.5 mm
- net Net-(D17-A1): track 18.5 -> 19.0 mm
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- added copper zone on F.Cu, net +3.3V
- added copper zone on F.Cu, net Net-(J4-In)
- added copper zone on F.Cu, net Net-(J8-In)
- added copper zone on F.Cu, net Net-(U6-LNA_IN)
- added copper zone on F.Cu, net Net-(U8-RFC)
