File: Node_F4_V.1.6.kicad_pcb (KiCad board)
At the start: 2 copper layers, 97.5 x 59 mm, 178 parts, among them IC2 MP1584EN, J1 Conn_Jack-DC, J2 Conn_01x10, J3 Conn_01x16_Female, J4 RF_IPEX_U.FL-R-SMT, J5 SWD, J6 WiFi_Prog, J7 RS485, J8 LoRa_Anten, Q1 P_Mosfet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

Commit message: Sua day cong
Parts:
- turned G1 to 90 degrees
Routing:
- net /I2C_SDA: track 23.8 -> 31.3 mm
- net /I2C_SCL: track 21.7 -> 28.7 mm
- net +3.3V: track 503.5 -> 499.8 mm, vias 25 -> 27
- net Net-(U3-NRST): track 58.8 -> 61.2 mm
- net /ESP_RX_LOAD: track 37.5 -> 38.8 mm
- net /ESP_TX_LOAD: track 40.2 -> 41.4 mm
- net Net-(U6-GPIO16): track 34.8 -> 34.1 mm
- net /UART_TX_LOG: track 17.7 -> 18.4 mm
- net GND: vias 196 -> 492
Other:
- board text added: "DESIGNED BY TRAN DINH HOANG ANH 20139061 MAI VAN ANH 20139059"

Commit message: Layout flash ESP32
Parts:
- moved C57 5.67 mm to (93.1, 86.6), turned to 0 degrees
- moved U4 2.16 mm to (99.3, 84.6), turned to 180 degrees
- moved BT1 0.28 mm to (88.8, 95.7)
- moved C47 0.18 mm to (94.6, 80.7)
Routing:
- net /SWP_SD3: track 21.7 -> 13.0 mm, vias 0 -> 2
- net Net-(U4-VCC): track 13.2 -> 7.80 mm
- net /SHD_SD2: track 11.3 -> 6.11 mm, vias 2 -> 0
- net /SCK_CLK: track 6.58 -> 4.76 mm
- net Net-(U6-GPIO16): track 34.1 -> 35.3 mm
- net +3.3V: track 499.8 -> 501.0 mm
- net /SCS_CMD: track 15.5 -> 14.5 mm
- net GND: vias 492 -> 478
Other:
- board size 97.5 x 59 mm -> 98 x 59 mm
- board text added: "BUCK MP1584"
- board text added: "RS485 SP3485"
- board text removed: "SP3485"

Commit message: LAYOUT OK check schematic again
Parts:
- moved C27 0.46 mm to (129.3, 90.8)
Routing:
- net +3.3V: track 501.0 -> 503.9 mm
- net /LORA NSS: track 24.6 -> 25.3 mm
- net /SPI3_MOSI: track 24.4 -> 25.1 mm
- net /SPI3_MISO: track 24.5 -> 25.1 mm
- net /SPI3_SCK: track 24.2 -> 24.8 mm
- net GND: vias 478 -> 487
